Commit message: chore: update spider robot configuration, including urdf symmetry fixes, controller updates, and auto-stand script

File: dog2_description/urdf/dog2.urdf.xacro (robot description, xacro)
@@ -9,4 +9,6 @@
 -->
 <robot xmlns:xacro="http://www.ros.org/wiki/xacro" name="dog2">
+  <xacro:arg name="controllers_yaml" default="$(find dog2_description)/config/ros2_controllers.yaml"/>
+  <xacro:property name="controllers_yaml" value="$(arg controllers_yaml)"/>
   <!-- Joint limits -->
   <xacro:property name="hip_lower_limit" value="-2.618"/>
@@ -56,6 +58,10 @@
     </collision>
   </link>
+  <xacro:property name="l1_inertia_xyz" value="-0.0159999123716776 0.000737036465389251 0.0261570925915838"/>
+  <xacro:property name="l2_inertia_xyz" value="0.0159999123716776 0.000737036465389251 0.0261570925915838"/>
+  <xacro:property name="l3_inertia_xyz" value="-0.0159999123716776 0.000737036465389251 0.0261570925915838"/>
+  <xacro:property name="l4_inertia_xyz" value="0.0159999123716776 0.000737036465389251 0.0261570925915838"/>
   <!-- Leg macro -->
-  <xacro:macro name="leg" params="prefix leg_num xyz rpy p_low p_up thigh_xyz shin_xyz
+  <xacro:macro name="leg" params="prefix leg_num xyz rpy p_low p_up thigh_xyz shin_xyz slider_inertia_xyz
                                  hip_rpy:='0 0 1.5708' hip_xyz:='-0.016 0.0199 0.055'
                                  knee_xyz:='-0.0233 -0.055 0.0274'
@@ -63,5 +69,5 @@
   <link name="l${leg_num}">
     <inertial>
-      <origin rpy="0 0 0" xyz="-0.0159999123716776 0.000737036465389251 0.0261570925915838"/>
+      <origin rpy="0 0 0" xyz="${slider_inertia_xyz}"/>
       <mass value="0.3"/>
       <inertia ixx="0.000107100908138004" ixy="0" ixz="0" iyy="8.38648309010005E-05" iyz="0" izz="7.86994452918461E-05"/>
@@ -189,13 +195,13 @@
   <!-- Leg instantiations -->
   <xacro:leg prefix="lf" leg_num="1" xyz="1.1026 -0.80953 0.2649" rpy="1.5708 0 0" p_low="-0.111" p_up="0.0"
-             thigh_xyz="${leg12_thigh_xyz}" shin_xyz="${leg12_shin_xyz}"/>
+             thigh_xyz="${leg12_thigh_xyz}" shin_xyz="${leg12_shin_xyz}" slider_inertia_xyz="${l1_inertia_xyz}"/>
   <xacro:leg prefix="rf" leg_num="2" xyz="1.3491 -0.80953 0.2649" rpy="1.5708 0 0" p_low="0.0" p_up="0.111"
-             thigh_xyz="${leg12_thigh_xyz}" shin_xyz="${leg12_shin_xyz}"
+             thigh_xyz="${leg12_thigh_xyz}" shin_xyz="${leg12_shin_xyz}" slider_inertia_xyz="${l2_inertia_xyz}"
              hip_xyz="0.016 0.0199 0.055"/>
   <xacro:leg prefix="lh" leg_num="3" xyz="1.3491 -0.68953 0.2649" rpy="1.5708 0 -3.1416" p_low="-0.111" p_up="0.0"
-             thigh_xyz="${leg3_thigh_xyz}" shin_xyz="${leg3_shin_xyz}"
+             thigh_xyz="${leg3_thigh_xyz}" shin_xyz="${leg3_shin_xyz}" slider_inertia_xyz="${l3_inertia_xyz}"
              hip_rpy="3.1416 0 1.5708" knee_xyz="-0.0233 -0.055 -0.0254"/>
   <xacro:leg prefix="rh" leg_num="4" xyz="1.1071 -0.68953 0.2649" rpy="1.5708 0 -3.1416" p_low="0.0" p_up="0.111"
-             thigh_xyz="${leg4_thigh_xyz}" shin_xyz="${leg4_shin_xyz}"
+             thigh_xyz="${leg4_thigh_xyz}" shin_xyz="${leg4_shin_xyz}" slider_inertia_xyz="${l4_inertia_xyz}"
              hip_rpy="3.1416 0 1.5708" hip_xyz="0.0116 0.0199 0.055" knee_xyz="-0.0233 -0.055 -0.0254"
              thigh_rpy="0 3.1416 0" thigh_col_rpy="0 3.1416 0"/>
@@ -288,5 +294,5 @@
   <gazebo>
     <plugin filename="libgazebo_ros2_control.so" name="gazebo_ros2_control">
-      <parameters>$(find dog2_description)/config/ros2_controllers.yaml</parameters>
+      <parameters>${controllers_yaml}</parameters>
       <robot_param>robot_description</robot_param>
       <robot_param_node>robot_state_publisher</robot_param_node>

Commit message: refactor: unify leg coordinate systems to Z-up and simplify joint axis definitions

File: dog2_description/urdf/dog2.urdf.xacro (robot description, xacro)
@@ -64,5 +64,5 @@
   <!-- Leg macro -->
   <xacro:macro name="leg" params="prefix leg_num xyz rpy p_low p_up thigh_xyz shin_xyz slider_inertia_xyz
-                                 hip_rpy:='0 0 1.5708' hip_xyz:='-0.016 0.0199 0.055'
+                                 hip_rpy:='0 0 0' hip_xyz:='-0.016 0.0199 0.055'
                                  knee_xyz:='-0.0233 -0.055 0.0274'
                                  thigh_rpy:='0 0 0' thigh_col_rpy:='0 0 0'">
@@ -122,5 +122,5 @@
     <parent link="l${leg_num}"/>
     <child link="${prefix}_hip_link"/>
-    <axis xyz="-1 0 0"/>
+    <axis xyz="0 0 1"/>
     <limit effort="${hip_effort}" lower="${hip_lower_limit}" upper="${hip_upper_limit}" velocity="${hip_velocity}"/>
   </joint>
@@ -148,8 +148,8 @@
   </link>
   <joint name="${prefix}_hfe_joint" type="revolute">
-    <origin rpy="1.5708 1.5708 0" xyz="${knee_xyz}"/>
+    <origin rpy="1.5708 0 0" xyz="${knee_xyz}"/>
     <parent link="${prefix}_hip_link"/>
     <child link="${prefix}_upper_leg_link"/>
-    <axis xyz="-1 0 0"/>
+    <axis xyz="0 0 1"/>
     <limit effort="${knee_effort}" lower="${knee_lower_limit}" upper="${knee_upper_limit}" velocity="${knee_velocity}"/>
   </joint>
@@ -180,5 +180,5 @@
     <parent link="${prefix}_upper_leg_link"/>
     <child link="${prefix}_lower_leg_link"/>
-    <axis xyz="-1 0 0"/>
+    <axis xyz="0 0 1"/>
     <limit effort="${knee_effort}" lower="${knee_lower_limit}" upper="${knee_upper_limit}" velocity="${knee_velocity}"/>
   </joint>
@@ -194,15 +194,16 @@
   </xacro:macro>
   <!-- Leg instantiations -->
-  <xacro:leg prefix="lf" leg_num="1" xyz="1.1026 -0.80953 0.2649" rpy="1.5708 0 0" p_low="-0.111" p_up="0.0"
-             thigh_xyz="${leg12_thigh_xyz}" shin_xyz="${leg12_shin_xyz}" slider_inertia_xyz="${l1_inertia_xyz}"/>
-  <xacro:leg prefix="rf" leg_num="2" xyz="1.3491 -0.80953 0.2649" rpy="1.5708 0 0" p_low="0.0" p_up="0.111"
+  <xacro:leg prefix="lf" leg_num="1" xyz="1.1026 -0.80953 0.2649" rpy="0 0 0" p_low="-0.111" p_up="0.0"
+             thigh_xyz="${leg12_thigh_xyz}" shin_xyz="${leg12_shin_xyz}" slider_inertia_xyz="${l1_inertia_xyz}"
+             hip_rpy="0 0 0"/>
+  <xacro:leg prefix="rf" leg_num="2" xyz="1.3491 -0.80953 0.2649" rpy="0 0 3.1416" p_low="0.0" p_up="0.111"
              thigh_xyz="${leg12_thigh_xyz}" shin_xyz="${leg12_shin_xyz}" slider_inertia_xyz="${l2_inertia_xyz}"
-             hip_xyz="0.016 0.0199 0.055"/>
-  <xacro:leg prefix="lh" leg_num="3" xyz="1.3491 -0.68953 0.2649" rpy="1.5708 0 -3.1416" p_low="-0.111" p_up="0.0"
+             hip_xyz="0.016 0.0199 0.055" hip_rpy="0 0 0"/>
+  <xacro:leg prefix="lh" leg_num="3" xyz="1.3491 -0.68953 0.2649" rpy="0 0 0" p_low="-0.111" p_up="0.0"
              thigh_xyz="${leg3_thigh_xyz}" shin_xyz="${leg3_shin_xyz}" slider_inertia_xyz="${l3_inertia_xyz}"
-             hip_rpy="3.1416 0 1.5708" knee_xyz="-0.0233 -0.055 -0.0254"/>
-  <xacro:leg prefix="rh" leg_num="4" xyz="1.1071 -0.68953 0.2649" rpy="1.5708 0 -3.1416" p_low="0.0" p_up="0.111"
+             hip_rpy="0 0 3.1416" knee_xyz="-0.0233 -0.055 -0.0254"/>
+  <xacro:leg prefix="rh" leg_num="4" xyz="1.1071 -0.68953 0.2649" rpy="0 0 3.1416" p_low="0.0" p_up="0.111"
              thigh_xyz="${leg4_thigh_xyz}" shin_xyz="${leg4_shin_xyz}" slider_inertia_xyz="${l4_inertia_xyz}"
-             hip_rpy="3.1416 0 1.5708" hip_xyz="0.0116 0.0199 0.055" knee_xyz="-0.0233 -0.055 -0.0254"
+             hip_rpy="0 0 3.1416" hip_xyz="0.0116 0.0199 0.055" knee_xyz="-0.0233 -0.055 -0.0254"
              thigh_rpy="0 3.1416 0" thigh_col_rpy="0 3.1416 0"/>
   <!-- ROS 2 Control -->

Commit message: revert: restore original mirrored coordinate system and update spider stand pose

File: dog2_description/urdf/dog2.urdf.xacro (robot description, xacro)
@@ -64,5 +64,5 @@
   <!-- Leg macro -->
   <xacro:macro name="leg" params="prefix leg_num xyz rpy p_low p_up thigh_xyz shin_xyz slider_inertia_xyz
-                                 hip_rpy:='0 0 0' hip_xyz:='-0.016 0.0199 0.055'
+                                 hip_rpy:='0 0 1.5708' hip_xyz:='-0.016 0.0199 0.055'
                                  knee_xyz:='-0.0233 -0.055 0.0274'
                                  thigh_rpy:='0 0 0' thigh_col_rpy:='0 0 0'">
@@ -122,5 +122,5 @@
     <parent link="l${leg_num}"/>
     <child link="${prefix}_hip_link"/>
-    <axis xyz="0 0 1"/>
+    <axis xyz="-1 0 0"/>
     <limit effort="${hip_effort}" lower="${hip_lower_limit}" upper="${hip_upper_limit}" velocity="${hip_velocity}"/>
   </joint>
@@ -148,8 +148,8 @@
   </link>
   <joint name="${prefix}_hfe_joint" type="revolute">
-    <origin rpy="1.5708 0 0" xyz="${knee_xyz}"/>
+    <origin rpy="1.5708 1.5708 0" xyz="${knee_xyz}"/>
     <parent link="${prefix}_hip_link"/>
     <child link="${prefix}_upper_leg_link"/>
-    <axis xyz="0 0 1"/>
+    <axis xyz="-1 0 0"/>
     <limit effort="${knee_effort}" lower="${knee_lower_limit}" upper="${knee_upper_limit}" velocity="${knee_velocity}"/>
   </joint>
@@ -180,5 +180,5 @@
     <parent link="${prefix}_upper_leg_link"/>
     <child link="${prefix}_lower_leg_link"/>
-    <axis xyz="0 0 1"/>
+    <axis xyz="-1 0 0"/>
     <limit effort="${knee_effort}" lower="${knee_lower_limit}" upper="${knee_upper_limit}" velocity="${knee_velocity}"/>
   </joint>
@@ -194,16 +194,15 @@
   </xacro:macro>
   <!-- Leg instantiations -->
-  <xacro:leg prefix="lf" leg_num="1" xyz="1.1026 -0.80953 0.2649" rpy="0 0 0" p_low="-0.111" p_up="0.0"
-             thigh_xyz="${leg12_thigh_xyz}" shin_xyz="${leg12_shin_xyz}" slider_inertia_xyz="${l1_inertia_xyz}"
-             hip_rpy="0 0 0"/>
-  <xacro:leg prefix="rf" leg_num="2" xyz="1.3491 -0.80953 0.2649" rpy="0 0 3.1416" p_low="0.0" p_up="0.111"
+  <xacro:leg prefix="lf" leg_num="1" xyz="1.1026 -0.80953 0.2649" rpy="1.5708 0 0" p_low="-0.111" p_up="0.0"
+             thigh_xyz="${leg12_thigh_xyz}" shin_xyz="${leg12_shin_xyz}" slider_inertia_xyz="${l1_inertia_xyz}"/>
+  <xacro:leg prefix="rf" leg_num="2" xyz="1.3491 -0.80953 0.2649" rpy="1.5708 0 0" p_low="0.0" p_up="0.111"
              thigh_xyz="${leg12_thigh_xyz}" shin_xyz="${leg12_shin_xyz}" slider_inertia_xyz="${l2_inertia_xyz}"
-             hip_xyz="0.016 0.0199 0.055" hip_rpy="0 0 0"/>
-  <xacro:leg prefix="lh" leg_num="3" xyz="1.3491 -0.68953 0.2649" rpy="0 0 0" p_low="-0.111" p_up="0.0"
+             hip_xyz="0.016 0.0199 0.055"/>
+  <xacro:leg prefix="lh" leg_num="3" xyz="1.3491 -0.68953 0.2649" rpy="1.5708 0 -3.1416" p_low="-0.111" p_up="0.0"
              thigh_xyz="${leg3_thigh_xyz}" shin_xyz="${leg3_shin_xyz}" slider_inertia_xyz="${l3_inertia_xyz}"
-             hip_rpy="0 0 3.1416" knee_xyz="-0.0233 -0.055 -0.0254"/>
-  <xacro:leg prefix="rh" leg_num="4" xyz="1.1071 -0.68953 0.2649" rpy="0 0 3.1416" p_low="0.0" p_up="0.111"
+             hip_rpy="3.1416 0 1.5708" knee_xyz="-0.0233 -0.055 -0.0254"/>
+  <xacro:leg prefix="rh" leg_num="4" xyz="1.1071 -0.68953 0.2649" rpy="1.5708 0 -3.1416" p_low="0.0" p_up="0.111"
              thigh_xyz="${leg4_thigh_xyz}" shin_xyz="${leg4_shin_xyz}" slider_inertia_xyz="${l4_inertia_xyz}"
-             hip_rpy="0 0 3.1416" hip_xyz="0.0116 0.0199 0.055" knee_xyz="-0.0233 -0.055 -0.0254"
+             hip_rpy="3.1416 0 1.5708" hip_xyz="0.0116 0.0199 0.055" knee_xyz="-0.0233 -0.055 -0.0254"
              thigh_rpy="0 3.1416 0" thigh_col_rpy="0 3.1416 0"/>
   <!-- ROS 2 Control -->
