Commit message: Sync dog2 description, prefixed meshes, and motion-control stack
Restore the dog2_description package layout with lf/lh/rh/rf mesh assets,
extend dog2.urdf.xacro with foot_link debug spheres and foot_fixed origins,
and align dog2_motion_control (joint names, leg parameters, kinematics,
tests, and new launch and utility modules). Update DEVELOPMENT_LOG and
visualization packaging.

Made-with: Cursor

File: src/dog2_description/urdf/dog2.urdf.xacro (robot description, xacro)
@@ -22,12 +22,4 @@
   <xacro:property name="prismatic_effort" value="100"/>
   <xacro:property name="prismatic_velocity" value="5"/>
-  <!--
-    Simulation mass scaling factor for A/B testing.
-    Set to 1.0 for normal operation.
-    For the "divide by 4" comparison run, set to 0.25.
-    This value is provided by the URDF xacro launch mapping.
-  -->
-  <xacro:arg name="mass_scale" default="1.0"/>
-  <xacro:property name="mass_scale" value="$(arg mass_scale)"/>
   <!-- Shared angle constants -->
   <xacro:property name="PI_CONST" value="3.141592653589793"/>
@@ -54,4 +46,14 @@
   <xacro:property name="leg4_thigh_xyz" value="-0.026 -0.0760041259902766 0.0649874821212069"/>
   <xacro:property name="leg4_shin_xyz" value="-0.0265089672547710 -0.1429895138560395 -0.0691152554666486"/>
+  <!--
+    foot_tip_xyz (tibia_link frame): *_foot_fixed / 绿色调试球心位置（回退前工作区基准）。
+    YZ: L3 沿胫骨在 YZ 平面内方向；X: 向机身横向收拢（foot_tip_lateral_inboard_m）。
+    Z: foot_tip_z_down_m 为沿 -tibia Z 的累计下调量（球 r=0.012）；与 leg_parameters.FOOT_TIP_* 保持一致。
+  -->
+  <xacro:property name="foot_tip_lateral_inboard_m" value="0.024"/>
+  <xacro:property name="foot_tip_z_down_m" value="0.012"/>
+  <xacro:property name="leg12_foot_tip_xyz" value="${foot_tip_lateral_inboard_m} -0.269179 -0.142168"/>
+  <xacro:property name="leg3_foot_tip_xyz" value="-${foot_tip_lateral_inboard_m} -0.269179 -0.142168"/>
+  <xacro:property name="leg4_foot_tip_xyz" value="-${foot_tip_lateral_inboard_m} -0.269202 -0.142121"/>
   <!-- World and base -->
   <link name="base_footprint"/>
@@ -84,6 +86,6 @@
     <inertial>
       <origin xyz="0.2492 0.12503 0.0" rpy="${half_pi} 0 0"/>
-      <mass value="${mass_scale * 6.0}"/>
-      <inertia ixx="${mass_scale * 0.0153}" ixy="${mass_scale * 0.00011}" ixz="0" iyy="${mass_scale * 0.052}" iyz="0" izz="${mass_scale * 0.044}"/>
+      <mass value="6.0"/>
+      <inertia ixx="0.0153" ixy="0.00011" ixz="0" iyy="0.052" iyz="0" izz="0.044"/>
     </inertial>
     <visual>
@@ -108,5 +110,5 @@
   <xacro:property name="l4_inertia_xyz" value="0.0159999123716776 0.000737036465389251 0.0261570925915838"/>
   <!-- Leg macro -->
-  <xacro:macro name="leg" params="prefix leg_num xyz_x xyz_y xyz_z rpy p_low p_up thigh_xyz shin_xyz slider_inertia_xyz
+  <xacro:macro name="leg" params="prefix leg_num xyz_x xyz_y xyz_z rpy p_low p_up thigh_xyz shin_xyz slider_inertia_xyz foot_tip_xyz
                                  hip_rpy:='0 0 ${half_pi}' hip_xyz:='-0.016 0.0199 0.055'
                                  knee_xyz:='-0.0233 -0.055 0.0274'
@@ -115,6 +117,6 @@
     <inertial>
       <origin rpy="0 0 0" xyz="${slider_inertia_xyz}"/>
-      <mass value="${mass_scale * 0.3}"/>
-      <inertia ixx="${mass_scale * 0.0001071}" ixy="0" ixz="0" iyy="${mass_scale * 8.386e-05}" iyz="0" izz="${mass_scale * 7.869e-05}"/>
+      <mass value="0.3"/>
+      <inertia ixx="0.0001071" ixy="0" ixz="0" iyy="8.386e-05" iyz="0" izz="7.869e-05"/>
     </inertial>
     <visual>
@@ -141,6 +143,6 @@
     <inertial>
       <origin rpy="0 0 0" xyz="-0.0233 -0.0383 0.000879"/>
-      <mass value="${mass_scale * 0.25}"/>
-      <inertia ixx="${mass_scale * 0.0001}" ixy="0" ixz="0" iyy="${mass_scale * 0.0001}" iyz="0" izz="${mass_scale * 0.0001}"/>
+      <mass value="0.25"/>
+      <inertia ixx="0.0001" ixy="0" ixz="0" iyy="0.0001" iyz="0" izz="0.0001"/>
     </inertial>
     <visual>
@@ -167,6 +169,6 @@
     <inertial>
       <origin rpy="0 0 0" xyz="${thigh_xyz}"/>
-      <mass value="${mass_scale * 0.4}"/>
-      <inertia ixx="${mass_scale * 0.000666}" ixy="0" ixz="0" iyy="${mass_scale * 0.000356}" iyz="${mass_scale * 0.000266}" izz="${mass_scale * 0.000534}"/>
+      <mass value="0.4"/>
+      <inertia ixx="0.000666" ixy="0" ixz="0" iyy="0.000356" iyz="0.000266" izz="0.000534"/>
     </inertial>
     <visual>
@@ -195,6 +197,6 @@
     <inertial>
       <origin rpy="0 0 0" xyz="${shin_xyz}"/>
-      <mass value="${mass_scale * 0.5}"/>
-      <inertia ixx="${mass_scale * 0.004517}" ixy="${mass_scale * 0.0000087}" ixz="${mass_scale * 0.0000042}" iyy="${mass_scale * 0.000975}" iyz="${mass_scale * -0.001769}" izz="${mass_scale * 0.003666}"/>
+      <mass value="0.5"/>
+      <inertia ixx="0.004517" ixy="0.0000087" ixz="0.0000042" iyy="0.000975" iyz="-0.001769" izz="0.003666"/>
     </inertial>
     <visual>
@@ -218,8 +220,24 @@
     <dynamics damping="${knee_damping}" friction="${knee_friction}"/>
   </joint>
-  <!--
-    Contact is currently attached to tibia as foot proxy.
-    TODO: split dedicated foot link/contact surface when available.
-  -->
+  <joint name="${prefix}_foot_fixed" type="fixed">
+    <origin rpy="0 0 0" xyz="${foot_tip_xyz}"/>
+    <parent link="${prefix}_tibia_link"/>
+    <child link="${prefix}_foot_link"/>
+  </joint>
+  <!-- foot_link: 足端坐标系 + 绿色小球 visual（调试用）。主碰撞仍在 tibia_link mesh。 -->
+  <link name="${prefix}_foot_link">
+    <inertial>
+      <origin rpy="0 0 0" xyz="0 0 0"/>
+      <mass value="0.04"/>
+      <inertia ixx="2.30e-06" ixy="0" ixz="0" iyy="2.30e-06" iyz="0" izz="2.30e-06"/>
+    </inertial>
+    <visual>
+      <origin rpy="0 0 0" xyz="0 0 0"/>
+      <geometry>
+        <sphere radius="0.012"/>
+      </geometry>
+      <material name="mat_foot_debug"><color rgba="0.2 0.85 0.35 1"/></material>
+    </visual>
+  </link>
   <gazebo reference="${prefix}_tibia_link">
     <mu1>${foot_contact_mu1}</mu1>
@@ -242,18 +260,22 @@
   <!-- Leg 1: Front Left (lf) base_link-local anchor -->
   <xacro:leg prefix="lf" leg_num="1" xyz_x="0.1246" xyz_y="0.0625" xyz_z="0.0" rpy="${half_pi} 0 0" p_low="-0.111" p_up="0.0"
-             thigh_xyz="${leg12_thigh_xyz}" shin_xyz="${leg12_shin_xyz}" slider_inertia_xyz="${l1_inertia_xyz}"/>
+             thigh_xyz="${leg12_thigh_xyz}" shin_xyz="${leg12_shin_xyz}" slider_inertia_xyz="${l1_inertia_xyz}"
+             foot_tip_xyz="${leg12_foot_tip_xyz}"/>
   <!-- Leg 2: Rear Left (lh) base_link-local anchor -->
   <xacro:leg prefix="lh" leg_num="2" xyz_x="0.3711" xyz_y="0.0625" xyz_z="0.0" rpy="${half_pi} 0 0" p_low="0.0" p_up="0.111"
              thigh_xyz="${leg12_thigh_xyz}" shin_xyz="${leg12_shin_xyz}" slider_inertia_xyz="${l2_inertia_xyz}"
-             hip_xyz="0.016 0.0199 0.055"/>
+             hip_xyz="0.016 0.0199 0.055"
+             foot_tip_xyz="${leg12_foot_tip_xyz}"/>
   <!-- Leg 3: Rear Right (rh) base_link-local anchor -->
   <xacro:leg prefix="rh" leg_num="3" xyz_x="0.3711" xyz_y="0.1825" xyz_z="0.0" rpy="${half_pi} 0 ${-pi}" p_low="-0.111" p_up="0.0"
              thigh_xyz="${leg3_thigh_xyz}" shin_xyz="${leg3_shin_xyz}" slider_inertia_xyz="${l3_inertia_xyz}"
-             hip_rpy="${pi} 0 ${half_pi}" knee_xyz="-0.0233 -0.055 -0.0254"/>
+             hip_rpy="${pi} 0 ${half_pi}" knee_xyz="-0.0233 -0.055 -0.0254"
+             foot_tip_xyz="${leg3_foot_tip_xyz}"/>
   <!-- Leg 4: Front Right (rf) base_link-local anchor -->
   <xacro:leg prefix="rf" leg_num="4" xyz_x="0.1291" xyz_y="0.1825" xyz_z="0.0" rpy="${half_pi} 0 ${-pi}" p_low="0.0" p_up="0.111"
              thigh_xyz="${leg4_thigh_xyz}" shin_xyz="${leg4_shin_xyz}" slider_inertia_xyz="${l4_inertia_xyz}"
              hip_rpy="${pi} 0 ${half_pi}" hip_xyz="0.0116 0.0199 0.055" knee_xyz="-0.0233 -0.055 -0.0254"
-             thigh_rpy="0 ${pi} 0" thigh_col_rpy="0 ${pi} 0"/>
+             thigh_rpy="0 ${pi} 0" thigh_col_rpy="0 ${pi} 0"
+             foot_tip_xyz="${leg4_foot_tip_xyz}"/>
   <!-- ROS 2 Control -->
   <ros2_control name="GazeboSimSystem" type="system">
@@ -345,7 +367,4 @@
     <plugin filename="libgz_ros2_control-system.so" name="gz_ros2_control::GazeboSimROS2ControlPlugin">
       <parameters>${controllers_yaml}</parameters>
-      <!-- Keep consistent with ros2_controllers.yaml (gz_ros_control.ros__parameters.*). -->
-      <hold_joints>true</hold_joints>
-      <position_proportional_gain>1.0</position_proportional_gain>
       <robot_param>robot_description</robot_param>
       <robot_param_node>robot_state_publisher</robot_param_node>

Commit message: feat(urdf): 足端 foot_link 闭环、原语碰撞、GZ 接触与 MPC 桥接
- foot_link: 球碰撞/惯量、摩擦与 contact sensor；胫骨 box + 低摩擦 Gazebo
- base/tibia 碰撞改为与 STL AABB 对齐的 box
- xacro 左右镜像常量；ros2_control 同时暴露 position 与 effort
- MPC 可选 GZ 足端接触；mpc launch 桥接与 spawn 碰撞高度支持 box/sphere
- DEVELOPMENT_LOG 2026-04-11 16:31 对话归档

File: src/dog2_description/urdf/dog2.urdf.xacro (robot description, xacro)
@@ -25,4 +25,10 @@
   <xacro:property name="PI_CONST" value="3.141592653589793"/>
   <xacro:property name="half_pi" value="1.5707963267948966"/>
+  <!-- 左右腿镜像：rail / 右侧髋关节 / 右侧膝几何 由常量表达，单腿仅保留必要不对称（如 hip_xyz、大腿 mesh 翻转）。 -->
+  <xacro:property name="leg_rail_rpy_L" value="${half_pi} 0 0"/>
+  <xacro:property name="leg_rail_rpy_R" value="${half_pi} 0 ${-PI_CONST}"/>
+  <xacro:property name="leg_hip_rpy_R" value="${PI_CONST} 0 ${half_pi}"/>
+  <xacro:property name="leg_knee_xyz_R" value="-0.0233 -0.055 -0.0254"/>
+  <xacro:property name="leg_thigh_mesh_flip_rpy" value="0 ${PI_CONST} 0"/>
   <!-- Joint passive dynamics (simulation stabilization) -->
   <xacro:property name="prismatic_damping" value="0.25"/>
@@ -49,11 +55,20 @@
     foot_tip_xyz (tibia_link frame): *_foot_fixed / 绿色调试球心位置（回退前工作区基准）。
     YZ: L3 沿胫骨在 YZ 平面内方向；X: 向机身横向收拢（foot_tip_lateral_inboard_m）。
-    Z: foot_tip_z_down_m 为沿 -tibia Z 的累计下调量（球 r=0.012）；与 leg_parameters.FOOT_TIP_* 保持一致。
+    Y: +半直径（+r）后再沿 −tibia Y 平移 1.5×直径（=3r）；Z: foot_tip_z_down_m；与 leg_parameters 一致。
   -->
+  <xacro:property name="foot_sphere_radius" value="0.012"/>
+  <xacro:property name="foot_tip_plus_y_half_diameter_m" value="${foot_sphere_radius}"/>
+  <xacro:property name="foot_tip_minus_y_one_and_half_diameter_m" value="${3 * foot_sphere_radius}"/>
   <xacro:property name="foot_tip_lateral_inboard_m" value="0.024"/>
   <xacro:property name="foot_tip_z_down_m" value="0.012"/>
-  <xacro:property name="leg12_foot_tip_xyz" value="${foot_tip_lateral_inboard_m} -0.269179 -0.142168"/>
-  <xacro:property name="leg3_foot_tip_xyz" value="-${foot_tip_lateral_inboard_m} -0.269179 -0.142168"/>
-  <xacro:property name="leg4_foot_tip_xyz" value="-${foot_tip_lateral_inboard_m} -0.269202 -0.142121"/>
+  <xacro:property name="leg12_foot_tip_xyz" value="${foot_tip_lateral_inboard_m} ${foot_tip_plus_y_half_diameter_m - foot_tip_minus_y_one_and_half_diameter_m - 0.269179} -0.142168"/>
+  <xacro:property name="leg3_foot_tip_xyz" value="-${foot_tip_lateral_inboard_m} ${foot_tip_plus_y_half_diameter_m - foot_tip_minus_y_one_and_half_diameter_m - 0.269179} -0.142168"/>
+  <xacro:property name="leg4_foot_tip_xyz" value="-${foot_tip_lateral_inboard_m} ${foot_tip_plus_y_half_diameter_m - foot_tip_minus_y_one_and_half_diameter_m - 0.269202} -0.142121"/>
+  <!-- base_link / tibia：与碰撞 STL AABB 对齐的 box 原语（数值接触更稳）。 -->
+  <xacro:property name="base_collision_box_size" value="0.342 0.16 0.1505"/>
+  <xacro:property name="base_collision_box_xyz" value="0.243 0.12247 0.01825"/>
+  <xacro:property name="tibia_collision_box_size" value="0.0508 0.31564 0.17558"/>
+  <xacro:property name="tibia_collision_box_xyz_L" value="0.0256 -0.14166 -0.07184"/>
+  <xacro:property name="tibia_collision_box_xyz_R" value="-0.0264 -0.14166 -0.07184"/>
   <!-- World and base -->
   <link name="base_footprint"/>
@@ -99,7 +114,7 @@
     </visual>
     <collision>
-      <origin xyz="-0.9780 0.87203 -0.2649" rpy="0 0 0"/>
-      <geometry>
-        <mesh filename="package://dog2_description/meshes/base_link.STL"/>
+      <origin xyz="${base_collision_box_xyz}" rpy="0 0 0"/>
+      <geometry>
+        <box size="${base_collision_box_size}"/>
       </geometry>
     </collision>
@@ -110,5 +125,5 @@
   <xacro:property name="l4_inertia_xyz" value="0.0159999123716776 0.000737036465389251 0.0261570925915838"/>
   <!-- Leg macro -->
-  <xacro:macro name="leg" params="prefix leg_num xyz_x xyz_y xyz_z rpy p_low p_up thigh_xyz shin_xyz slider_inertia_xyz foot_tip_xyz
+  <xacro:macro name="leg" params="prefix leg_num xyz_x xyz_y xyz_z rpy p_low p_up thigh_xyz shin_xyz slider_inertia_xyz foot_tip_xyz tibia_col_xyz
                                  hip_rpy:='0 0 ${half_pi}' hip_xyz:='-0.016 0.0199 0.055'
                                  knee_xyz:='-0.0233 -0.055 0.0274'
@@ -207,6 +222,7 @@
     </visual>
     <collision>
-      <geometry>
-        <mesh filename="package://dog2_description/meshes/collision/l${leg_num}111_collision.STL"/>
+      <origin rpy="0 0 0" xyz="${tibia_col_xyz}"/>
+      <geometry>
+        <box size="${tibia_collision_box_size}"/>
       </geometry>
     </collision>
@@ -225,20 +241,35 @@
     <child link="${prefix}_foot_link"/>
   </joint>
-  <!-- foot_link: 足端坐标系 + 绿色小球 visual（调试用）。主碰撞仍在 tibia_link mesh。 -->
+  <!-- foot_link: 足端 frame 原点 = 球心；collision 与 visual 同球（r=foot_sphere_radius）。 -->
   <link name="${prefix}_foot_link">
     <inertial>
       <origin rpy="0 0 0" xyz="0 0 0"/>
-      <mass value="0.04"/>
-      <inertia ixx="2.30e-06" ixy="0" ixz="0" iyy="2.30e-06" iyz="0" izz="2.30e-06"/>
+      <mass value="0.05"/>
+      <inertia ixx="2.88e-06" ixy="0" ixz="0" iyy="2.88e-06" iyz="0" izz="2.88e-06"/>
     </inertial>
     <visual>
       <origin rpy="0 0 0" xyz="0 0 0"/>
       <geometry>
-        <sphere radius="0.012"/>
+        <sphere radius="${foot_sphere_radius}"/>
       </geometry>
       <material name="mat_foot_debug"><color rgba="0.2 0.85 0.35 1"/></material>
     </visual>
-  </link>
+    <collision>
+      <origin rpy="0 0 0" xyz="0 0 0"/>
+      <geometry>
+        <sphere radius="${foot_sphere_radius}"/>
+      </geometry>
+    </collision>
+  </link>
+  <!-- 胫骨原语若蹭地：低刚度/低摩擦，主触地仍由 foot 球承担。 -->
   <gazebo reference="${prefix}_tibia_link">
+    <mu1>0.05</mu1>
+    <mu2>0.05</mu2>
+    <kp>800</kp>
+    <kd>8</kd>
+    <minDepth>${foot_contact_min_depth}</minDepth>
+    <maxVel>${foot_contact_max_vel}</maxVel>
+  </gazebo>
+  <gazebo reference="${prefix}_foot_link">
     <mu1>${foot_contact_mu1}</mu1>
     <mu2>${foot_contact_mu2}</mu2>
@@ -248,4 +279,9 @@
     <maxVel>${foot_contact_max_vel}</maxVel>
     <material>Gazebo/Grey</material>
+    <sensor name="${prefix}_foot_contact" type="contact">
+      <always_on>true</always_on>
+      <update_rate>200</update_rate>
+      <contact/>
+    </sensor>
   </gazebo>
   </xacro:macro>
@@ -259,23 +295,23 @@
   -->
   <!-- Leg 1: Front Left (lf) base_link-local anchor -->
-  <xacro:leg prefix="lf" leg_num="1" xyz_x="0.1246" xyz_y="0.0625" xyz_z="0.0" rpy="${half_pi} 0 0" p_low="-0.111" p_up="0.0"
+  <xacro:leg prefix="lf" leg_num="1" xyz_x="0.1246" xyz_y="0.0625" xyz_z="0.0" rpy="${leg_rail_rpy_L}" p_low="-0.111" p_up="0.0"
              thigh_xyz="${leg12_thigh_xyz}" shin_xyz="${leg12_shin_xyz}" slider_inertia_xyz="${l1_inertia_xyz}"
-             foot_tip_xyz="${leg12_foot_tip_xyz}"/>
+             foot_tip_xyz="${leg12_foot_tip_xyz}" tibia_col_xyz="${tibia_collision_box_xyz_L}"/>
   <!-- Leg 2: Rear Left (lh) base_link-local anchor -->
-  <xacro:leg prefix="lh" leg_num="2" xyz_x="0.3711" xyz_y="0.0625" xyz_z="0.0" rpy="${half_pi} 0 0" p_low="0.0" p_up="0.111"
+  <xacro:leg prefix="lh" leg_num="2" xyz_x="0.3711" xyz_y="0.0625" xyz_z="0.0" rpy="${leg_rail_rpy_L}" p_low="0.0" p_up="0.111"
              thigh_xyz="${leg12_thigh_xyz}" shin_xyz="${leg12_shin_xyz}" slider_inertia_xyz="${l2_inertia_xyz}"
              hip_xyz="0.016 0.0199 0.055"
-             foot_tip_xyz="${leg12_foot_tip_xyz}"/>
+             foot_tip_xyz="${leg12_foot_tip_xyz}" tibia_col_xyz="${tibia_collision_box_xyz_L}"/>
   <!-- Leg 3: Rear Right (rh) base_link-local anchor -->
-  <xacro:leg prefix="rh" leg_num="3" xyz_x="0.3711" xyz_y="0.1825" xyz_z="0.0" rpy="${half_pi} 0 ${-pi}" p_low="-0.111" p_up="0.0"
+  <xacro:leg prefix="rh" leg_num="3" xyz_x="0.3711" xyz_y="0.1825" xyz_z="0.0" rpy="${leg_rail_rpy_R}" p_low="-0.111" p_up="0.0"
              thigh_xyz="${leg3_thigh_xyz}" shin_xyz="${leg3_shin_xyz}" slider_inertia_xyz="${l3_inertia_xyz}"
-             hip_rpy="${pi} 0 ${half_pi}" knee_xyz="-0.0233 -0.055 -0.0254"
-             foot_tip_xyz="${leg3_foot_tip_xyz}"/>
+             hip_rpy="${leg_hip_rpy_R}" knee_xyz="${leg_knee_xyz_R}"
+             foot_tip_xyz="${leg3_foot_tip_xyz}" tibia_col_xyz="${tibia_collision_box_xyz_R}"/>
   <!-- Leg 4: Front Right (rf) base_link-local anchor -->
-  <xacro:leg prefix="rf" leg_num="4" xyz_x="0.1291" xyz_y="0.1825" xyz_z="0.0" rpy="${half_pi} 0 ${-pi}" p_low="0.0" p_up="0.111"
+  <xacro:leg prefix="rf" leg_num="4" xyz_x="0.1291" xyz_y="0.1825" xyz_z="0.0" rpy="${leg_rail_rpy_R}" p_low="0.0" p_up="0.111"
              thigh_xyz="${leg4_thigh_xyz}" shin_xyz="${leg4_shin_xyz}" slider_inertia_xyz="${l4_inertia_xyz}"
-             hip_rpy="${pi} 0 ${half_pi}" hip_xyz="0.0116 0.0199 0.055" knee_xyz="-0.0233 -0.055 -0.0254"
-             thigh_rpy="0 ${pi} 0" thigh_col_rpy="0 ${pi} 0"
-             foot_tip_xyz="${leg4_foot_tip_xyz}"/>
+             hip_rpy="${leg_hip_rpy_R}" hip_xyz="0.0116 0.0199 0.055" knee_xyz="${leg_knee_xyz_R}"
+             thigh_rpy="${leg_thigh_mesh_flip_rpy}" thigh_col_rpy="${leg_thigh_mesh_flip_rpy}"
+             foot_tip_xyz="${leg4_foot_tip_xyz}" tibia_col_xyz="${tibia_collision_box_xyz_R}"/>
   <!-- ROS 2 Control -->
   <ros2_control name="GazeboSimSystem" type="system">
@@ -285,4 +321,5 @@
     <joint name="lf_rail_joint">
       <command_interface name="position"/>
+      <command_interface name="effort"/>
       <state_interface name="position"/>
       <state_interface name="velocity"/>
@@ -290,4 +327,5 @@
     <joint name="lf_coxa_joint">
       <command_interface name="position"/>
+      <command_interface name="effort"/>
       <state_interface name="position"/>
       <state_interface name="velocity"/>
@@ -295,4 +333,5 @@
     <joint name="lf_femur_joint">
       <command_interface name="position"/>
+      <command_interface name="effort"/>
       <state_interface name="position"/>
       <state_interface name="velocity"/>
@@ -300,4 +339,5 @@
     <joint name="lf_tibia_joint">
       <command_interface name="position"/>
+      <command_interface name="effort"/>
       <state_interface name="position"/>
       <state_interface name="velocity"/>
@@ -305,4 +345,5 @@
     <joint name="lh_rail_joint">
       <command_interface name="position"/>
+      <command_interface name="effort"/>
       <state_interface name="position"/>
       <state_interface name="velocity"/>
@@ -310,4 +351,5 @@
     <joint name="lh_coxa_joint">
       <command_interface name="position"/>
+      <command_interface name="effort"/>
       <state_interface name="position"/>
       <state_interface name="velocity"/>
@@ -315,4 +357,5 @@
     <joint name="lh_femur_joint">
       <command_interface name="position"/>
+      <command_interface name="effort"/>
       <state_interface name="position"/>
       <state_interface name="velocity"/>
@@ -320,4 +363,5 @@
     <joint name="lh_tibia_joint">
       <command_interface name="position"/>
+      <command_interface name="effort"/>
       <state_interface name="position"/>
       <state_interface name="velocity"/>
@@ -325,4 +369,5 @@
     <joint name="rh_rail_joint">
       <command_interface name="position"/>
+      <command_interface name="effort"/>
       <state_interface name="position"/>
       <state_interface name="velocity"/>
@@ -330,4 +375,5 @@
     <joint name="rh_coxa_joint">
       <command_interface name="position"/>
+      <command_interface name="effort"/>
       <state_interface name="position"/>
       <state_interface name="velocity"/>
@@ -335,4 +381,5 @@
     <joint name="rh_femur_joint">
       <command_interface name="position"/>
+      <command_interface name="effort"/>
       <state_interface name="position"/>
       <state_interface name="velocity"/>
@@ -340,4 +387,5 @@
     <joint name="rh_tibia_joint">
       <command_interface name="position"/>
+      <command_interface name="effort"/>
       <state_interface name="position"/>
       <state_interface name="velocity"/>
@@ -345,4 +393,5 @@
     <joint name="rf_rail_joint">
       <command_interface name="position"/>
+      <command_interface name="effort"/>
       <state_interface name="position"/>
       <state_interface name="velocity"/>
@@ -350,4 +399,5 @@
     <joint name="rf_coxa_joint">
       <command_interface name="position"/>
+      <command_interface name="effort"/>
       <state_interface name="position"/>
       <state_interface name="velocity"/>
@@ -355,4 +405,5 @@
     <joint name="rf_femur_joint">
       <command_interface name="position"/>
+      <command_interface name="effort"/>
       <state_interface name="position"/>
       <state_interface name="velocity"/>
@@ -360,4 +411,5 @@
     <joint name="rf_tibia_joint">
       <command_interface name="position"/>
+      <command_interface name="effort"/>
       <state_interface name="position"/>
       <state_interface name="velocity"/>
