Commit message: chore: snapshot local crossing and locomotion updates

File: src/dog2_description/urdf/dog2.urdf.xacro (robot description, xacro)
@@ -59,4 +59,15 @@
   <xacro:property name="foot_contact_min_depth" value="0.0005"/>
   <xacro:property name="foot_contact_max_vel" value="0.2"/>
+  <!-- Tiny inertial block for massless frame-only links.
+       PyBullet assigns mass=1 kg to links with missing inertial data, which
+       makes these purely kinematic helper frames behave like heavy bodies in
+       dynamics. Keep this near-zero but nonzero so importers stay well-defined. -->
+  <xacro:macro name="frame_inertial" params="mass:=0.0001">
+    <inertial>
+      <origin xyz="0 0 0" rpy="0 0 0"/>
+      <mass value="${mass}"/>
+      <inertia ixx="1e-8" ixy="0" ixz="0" iyy="1e-8" iyz="0" izz="1e-8"/>
+    </inertial>
+  </xacro:macro>
   <!-- Inertia properties -->
   <xacro:property name="leg12_thigh_xyz" value="0.026 -0.0760041259902766 0.0649874821212071"/>
@@ -212,6 +223,10 @@
   <xacro:property name="coxa_joint_rpy_eff" value="0 0 0"/>
   <xacro:property name="coxa_axis_eff" value="0 0 -1"/>
-  <link name="${prefix}_coxa_axis_frame"/>
-  <link name="${prefix}_coxa_drive_frame"/>
+  <link name="${prefix}_coxa_axis_frame">
+    <xacro:frame_inertial/>
+  </link>
+  <link name="${prefix}_coxa_drive_frame">
+    <xacro:frame_inertial/>
+  </link>
   <joint name="${prefix}_coxa_axis_fixed" type="fixed">
     <parent link="${prefix}_rail_link"/>
@@ -283,6 +298,10 @@
   <xacro:property name="femur_joint_rpy_eff" value="${half_pi} ${half_pi} 0"/>
   <xacro:property name="femur_axis_eff" value="-1 0 0"/>
-  <link name="${prefix}_femur_axis_frame"/>
-  <link name="${prefix}_femur_drive_frame"/>
+  <link name="${prefix}_femur_axis_frame">
+    <xacro:frame_inertial/>
+  </link>
+  <link name="${prefix}_femur_drive_frame">
+    <xacro:frame_inertial/>
+  </link>
   <joint name="${prefix}_femur_axis_fixed" type="fixed">
     <parent link="${prefix}_coxa_link"/>
@@ -331,6 +350,10 @@
   <xacro:property name="tibia_joint_rpy_eff" value="0 0 0"/>
   <xacro:property name="tibia_axis_eff" value="-1 0 0"/>
-  <link name="${prefix}_tibia_axis_frame"/>
-  <link name="${prefix}_tibia_drive_frame"/>
+  <link name="${prefix}_tibia_axis_frame">
+    <xacro:frame_inertial/>
+  </link>
+  <link name="${prefix}_tibia_drive_frame">
+    <xacro:frame_inertial/>
+  </link>
   <joint name="${prefix}_tibia_axis_fixed" type="fixed">
     <parent link="${prefix}_femur_link"/>
@@ -411,5 +434,7 @@
   <!-- Leg instantiations -->
   <!-- Layering target: mount frames carry chassis asymmetry; the semantic chain stays parameterized. -->
-  <link name="lf_leg_mount"/>
+  <link name="lf_leg_mount">
+    <xacro:frame_inertial/>
+  </link>
   <joint name="lf_leg_mount_fixed" type="fixed">
     <parent link="base_link"/>
@@ -417,5 +442,7 @@
     <origin xyz="${0.1246 - base_link_semantic_origin_x} ${0.0625 - base_link_semantic_origin_y} ${0.0 - base_link_semantic_origin_z}" rpy="${leg_rail_rpy_L}"/>
   </joint>
-  <link name="lh_leg_mount"/>
+  <link name="lh_leg_mount">
+    <xacro:frame_inertial/>
+  </link>
   <joint name="lh_leg_mount_fixed" type="fixed">
     <parent link="base_link"/>
@@ -423,5 +450,7 @@
     <origin xyz="${0.3711 - base_link_semantic_origin_x} ${0.0625 - base_link_semantic_origin_y} ${0.0 - base_link_semantic_origin_z}" rpy="${leg_rail_rpy_L}"/>
   </joint>
-  <link name="rh_leg_mount"/>
+  <link name="rh_leg_mount">
+    <xacro:frame_inertial/>
+  </link>
   <joint name="rh_leg_mount_fixed" type="fixed">
     <parent link="base_link"/>
@@ -429,5 +458,7 @@
     <origin xyz="${0.3711 - base_link_semantic_origin_x} ${0.1825 - base_link_semantic_origin_y} ${0.0 - base_link_semantic_origin_z}" rpy="${leg_rail_rpy_R}"/>
   </joint>
-  <link name="rf_leg_mount"/>
+  <link name="rf_leg_mount">
+    <xacro:frame_inertial/>
+  </link>
   <joint name="rf_leg_mount_fixed" type="fixed">
     <parent link="base_link"/>
@@ -442,10 +473,10 @@
              hip_xyz="0.016 0.0199 0.055"
              foot_tip_xyz="${leg12_foot_tip_xyz}"/>
-  <xacro:leg prefix="rh" side="right" leg_num="3" parent_link="rh_leg_mount" rail_axis="${leg_rail_axis_R}" p_low="0.0" p_up="0.111"
+  <xacro:leg prefix="rh" side="right" leg_num="3" parent_link="rh_leg_mount" rail_axis="${leg_rail_axis_R}" p_low="-0.111" p_up="0.0"
              thigh_xyz="${leg3_thigh_xyz}" shin_xyz="${leg3_shin_xyz}" slider_inertia_xyz="${l3_inertia_xyz}"
              knee_xyz="${leg_knee_xyz_R}"
              foot_tip_xyz="${leg3_foot_tip_xyz}"/>
   <!-- Front-right retains its measured hip mount offset; the rest of the chain follows the shared contract. -->
-  <xacro:leg prefix="rf" side="right" leg_num="4" parent_link="rf_leg_mount" rail_axis="${leg_rail_axis_R}" p_low="-0.111" p_up="0.0"
+  <xacro:leg prefix="rf" side="right" leg_num="4" parent_link="rf_leg_mount" rail_axis="${leg_rail_axis_R}" p_low="0.0" p_up="0.111"
              thigh_xyz="${leg4_thigh_xyz}" shin_xyz="${leg4_shin_xyz}" slider_inertia_xyz="${l4_inertia_xyz}"
              hip_xyz="0.0116 0.0199 0.055" knee_xyz="${leg_knee_xyz_R}"
